Commit message: Support vertical doors

File: models/door.sdf.xacro (robot description, xacro)
@@ -4,6 +4,10 @@
   <xacro:arg name="type" default="slide"/>
   <xacro:arg name="direction" default="left"/>
+  <xacro:arg name="color" default="Green"/>
+  <xacro:arg name="axis" default="1 0 0"/>
+  <xacro:arg name="effort" default="10.0"/>
+  <xacro:arg name="velocity" default="1.0"/>
   <xacro:arg name="max_trans_dist" default="1.0"/>
-  <model name='sliding_door'>
+  <model name='door'>
     <link name='door'>
       <inertial>
@@ -19,5 +23,5 @@
         </inertia>
       </inertial>
-      <collision name='door_collision'>
+      <collision name='collision'>
         <pose>0 0 0 0 0 0</pose>
         <geometry>
@@ -35,5 +39,5 @@
         </surface>
       </collision>
-      <visual name='door_visual'>
+      <visual name='visual'>
         <pose>0 0 0 0 0 0</pose>
         <geometry>
@@ -44,5 +48,5 @@
         <material>
           <script>
-            <name>Gazebo/Green</name>
+            <name>Gazebo/$(arg color)</name>
             <uri>__default__</uri>
           </script>
@@ -56,14 +60,14 @@
       <self_collide>0</self_collide>
     </link>
-    <joint name='grounding_joint' type='prismatic'>
+    <joint name='door_joint' type='prismatic'>
       <child>door</child>
       <parent>world</parent>
       <axis>
-        <xyz>1 0 0</xyz>
+        <xyz>$(arg axis)</xyz>
         <limit>
           <lower>0</lower>
           <upper>-0.05</upper>
-          <effort>10</effort>
-          <velocity>0.5</velocity>
+          <effort>$(arg effort)</effort>
+          <velocity>$(arg velocity)</velocity>
         </limit>
         <dynamics>
